File: wiper.kicad_pcb (KiCad board)
At the start: 2 copper layers, 90 x 67.5 mm, 67 parts, among them J1 Conn_01x02, J10 Conn_01x02, J2 Sensor FW, J3 Sensor BK, J4 Conn_01x02, J5 Conn_01x02, J6 PROG, J7 I2C, J8 UART, J9 Conn_01x02, K1 G5LE-1, K2 G5LE-1, Q1 MMBT2222A, Q2 MMBT2222A, Q3 MMBT2222A, Q4 MMBT2222A, SW1 Reset, U1 LM7805_TO220, U2 PC817, U3 PC817, U4 KA78M05_TO252, U5 ATmega48-20A, Y1 16MHz

Commit message: v1.0: version sent to production (2026-02-11)
PCB matches the Gerber files generated 2026-02-11 18:12.
- Add potentiometer RV1 (10K) and capacitor C10 (100nF)
- Remove test point TP1
- Replace M3 ISO7380 mounting holes with M3
- Complete PCB routing

Schematic restored to its state at production time:
C7 = 100nF, matching the PCB.

Co-Authored-By: Claude Opus 5.5 <noreply@anthropic.com>
Claude-Session: https://claude.ai/code/session_01ADaCdURCPQ1EkJMwDbARyU
Parts:
- removed the REF** at (144.0, 56.0)
- removed the REF** at (223.0, 112.0)
- removed the REF** at (144.0, 112.0)
- removed the REF** at (223.0, 56.0)
- removed TP1: ~, Connector_PinHeader_1.00mm:PinHeader_1x01_P1.00mm_Vertical
- added C10: 100nF, Resistor_SMD:R_0603_1608Metric_Pad0.98x0.95mm_HandSolder, B.Cu at (172.8, 97.6)
- added REF**: MountingHole_3.2mm_M3, MountingHole:MountingHole_3.2mm_M3, F.Cu at (224.0, 113.0)
- added REF**: MountingHole_3.2mm_M3, MountingHole:MountingHole_3.2mm_M3, F.Cu at (224.0, 55.0)
- added REF**: MountingHole_3.2mm_M3, MountingHole:MountingHole_3.2mm_M3, F.Cu at (143.0, 113.0)
- added REF**: MountingHole_3.2mm_M3, MountingHole:MountingHole_3.2mm_M3, F.Cu at (143.0, 55.0)
- added RV1: 10K, Potentiometer_THT:Potentiometer_ACP_CA9-V10_Vertical, F.Cu at (170.3, 100.2)
- moved R4 6.40 mm to (164.4, 98.5)
- moved U3 6.40 mm to (164.3, 103.0)
- moved R2 5.55 mm to (170.0, 107.6), turned to 0 degrees
- moved Q4 2.71 mm to (187.0, 102.5)
- moved R14 2.71 mm to (184.2, 100.4)
- moved R16 2.71 mm to (187.0, 98.5)
- moved TP2 2.60 mm to (170.9, 90.2)
- moved J3 0.13 mm to (168.5, 110.9)
Routing:
- net ~: track 106.6 -> 200.3 mm, vias 3 -> 6
- net +24V: track 138.1 -> 206.1 mm
- net Net-(J10-Pin_2): track 22.4 -> 57.8 mm
- net Net-(K1-Pad3): track 51.3 -> 83.2 mm
- net Net-(K2-Pad3): track 25.8 -> 52.1 mm
- net Net-(J9-Pin_1): track 21.6 -> 45.8 mm
- net Net-(J10-Pin_1): track 20.2 -> 39.6 mm
- net Net-(J9-Pin_2): track 18.2 -> 37.4 mm
- net Net-(U5-ADC6): track 7.21 -> 19.2 mm, vias 0 -> 1
- net Net-(J3-Pin_2): track 13.8 -> 5.09 mm
- net Net-(R2-Pad1): track 2.59 -> 8.15 mm
- net /SENS_BK: track 19.8 -> 22.1 mm
- net Net-(D8-A): track 9.69 -> 7.65 mm
- net Net-(U5-ADC7): track 7.17 -> 6.04 mm
- net +5V: track 98.6 -> 99.5 mm
Other:
- board text added: "Reset"
- board text added: "Wiper ver. 2.2 05.02.2026"
- board text removed: "K"
- board text removed: "Wiper ver. 2.1 25.01.2026"
